File: hardware/core/core.kicad_pcb (KiCad board)
At the start: 2 copper layers, 0 parts

Commit message: Prompt is too long
Parts:
- added C1: 220n, Capacitor_THT:C_Rect_L7.0mm_W4.5mm_P5.00mm, F.Cu at (141.3, 63.6)
- added C2: 100n, Capacitor_THT:C_Rect_L7.0mm_W2.5mm_P5.00mm, F.Cu at (146.4, 63.7)
- added D1: 1N4148, Diode_THT:D_DO-35_SOD27_P7.62mm_Horizontal, B.Cu at (205.2, 156.2)
- added D10: 1N5817, Diode_THT:D_DO-41_SOD81_P10.16mm_Horizontal, F.Cu at (136.2, 58.4)
- added D2: 1N4148, Diode_THT:D_DO-35_SOD27_P7.62mm_Horizontal, B.Cu at (207.7, 156.2)
- added D3: 1N4148, Diode_THT:D_DO-35_SOD27_P7.62mm_Horizontal, B.Cu at (210.3, 156.2)
- added D4: 1N4148, Diode_THT:D_DO-35_SOD27_P7.62mm_Horizontal, B.Cu at (212.8, 156.2)
- added D5: 1N4148, Diode_THT:D_DO-35_SOD27_P7.62mm_Horizontal, B.Cu at (215.3, 156.2)
- added D6: 1N4148, Diode_THT:D_DO-35_SOD27_P7.62mm_Horizontal, B.Cu at (217.9, 156.2)
- added D7: 1N4148, Diode_THT:D_DO-35_SOD27_P7.62mm_Horizontal, B.Cu at (220.4, 156.2)
- added D8: 1N4148, Diode_THT:D_DO-35_SOD27_P7.62mm_Horizontal, B.Cu at (223.0, 156.2)
- added D9: 1N4148, Diode_THT:D_DO-35_SOD27_P7.62mm_Horizontal, F.Cu at (174.0, 73.7)
- added J1: 9V_IN, Connector_BarrelJack:BarrelJack_Horizontal, F.Cu at (127.0, 69.5)
- added J2: LCD, midilord:4004A, F.Cu at (203.2, 152.4)
- added J3: MIDI IN, DIN5_MIDI:DIN5_MIDI, F.Cu at (172.7, 67.3)
- added J4: MIDI OUT 1, DIN5_MIDI:DIN5_MIDI, F.Cu at (195.6, 67.3)
- added J5: MIDI OUT 2, Connector_Audio:Jack_6.35mm_Neutrik_NMJ6HFD2-AU_Horizontal, F.Cu at (213.4, 72.4)
- added J6: MIDI OUT 3, Connector_Audio:Jack_6.35mm_Neutrik_NMJ6HFD2-AU_Horizontal, F.Cu at (240.0, 72.4)
- added J7: MIDI OUT 4, Connector_Audio:Jack_6.35mm_Neutrik_NMJ6HFD2-AU_Horizontal, F.Cu at (266.7, 72.4)
- added R1: 220R, Resistor_THT:R_Axial_DIN0204_L3.6mm_D1.6mm_P7.62mm_Horizontal, F.Cu at (160.0, 73.7)
- added R10: 1K, Resistor_THT:R_Axial_DIN0204_L3.6mm_D1.6mm_P7.62mm_Horizontal, F.Cu at (152.4, 71.1)
- added R2: 33R, Resistor_THT:R_Axial_DIN0204_L3.6mm_D1.6mm_P7.62mm_Horizontal, F.Cu at (209.6, 67.3)
- added R3: 33R, Resistor_THT:R_Axial_DIN0204_L3.6mm_D1.6mm_P7.62mm_Horizontal, F.Cu at (236.2, 67.3)
- added R4: 33R, Resistor_THT:R_Axial_DIN0204_L3.6mm_D1.6mm_P7.62mm_Horizontal, F.Cu at (262.9, 67.3)
- added R5: 33R, Resistor_THT:R_Axial_DIN0204_L3.6mm_D1.6mm_P7.62mm_Horizontal, F.Cu at (196.8, 73.7)
- added R6: 10R, Resistor_THT:R_Axial_DIN0204_L3.6mm_D1.6mm_P7.62mm_Horizontal, F.Cu at (209.6, 57.1)
- added R7: 10R, Resistor_THT:R_Axial_DIN0204_L3.6mm_D1.6mm_P7.62mm_Horizontal, F.Cu at (236.2, 57.1)
- added R8: 10R, Resistor_THT:R_Axial_DIN0204_L3.6mm_D1.6mm_P7.62mm_Horizontal, F.Cu at (262.9, 57.1)
- added R9: 10R, Resistor_THT:R_Axial_DIN0204_L3.6mm_D1.6mm_P7.62mm_Horizontal, F.Cu at (194.3, 73.7)
- added RV1: 10K, Potentiometer_THT:Potentiometer_Bourns_3266W_Vertical, B.Cu at (109.2, 182.9)
- added SW1: FS, Connector_PinHeader_2.54mm:PinHeader_1x02_P2.54mm_Vertical, B.Cu at (128.3, 119.4)
- added SW2: FS, Connector_PinHeader_2.54mm:PinHeader_1x02_P2.54mm_Vertical, B.Cu at (128.3, 185.4)
- added SW3: FS, Connector_PinHeader_2.54mm:PinHeader_1x02_P2.54mm_Vertical, B.Cu at (179.1, 119.4)
- added SW4: FS, Connector_PinHeader_2.54mm:PinHeader_1x02_P2.54mm_Vertical, B.Cu at (179.1, 185.4)
- added SW5: FS, Connector_PinHeader_2.54mm:PinHeader_1x02_P2.54mm_Vertical, B.Cu at (229.9, 119.4)
- added SW6: FS, Connector_PinHeader_2.54mm:PinHeader_1x02_P2.54mm_Vertical, B.Cu at (229.9, 185.4)
- added SW7: FS, Connector_PinHeader_2.54mm:PinHeader_1x02_P2.54mm_Vertical, B.Cu at (280.7, 119.4)
- added SW8: FS, Connector_PinHeader_2.54mm:PinHeader_1x02_P2.54mm_Vertical, B.Cu at (280.7, 185.4)
- added U1: ESP32-S3-DevKitC, Espressif:ESP32-S3-DevKitC, B.Cu at (236.3, 141.0)
- added U2: L7805, Package_TO_SOT_THT:TO-220-3_Vertical, F.Cu at (141.3, 58.5)
- added U3: 6N137, Package_DIP:DIP-8_W7.62mm, F.Cu at (152.4, 59.7)
Routing:
- added copper zone on B.Cu, net GND
- added copper zone on F.Cu, net GND
Other:
- board outline added: 190.5 x 132.1 mm

Commit message: Prompt is too long
Parts:
- added C3: 100n, Capacitor_THT:C_Rect_L7.0mm_W2.5mm_P5.00mm, B.Cu at (101.6, 116.8)
- added C4: 100u, Capacitor_THT:CP_Radial_D8.0mm_P3.50mm, B.Cu at (94.0, 128.3)
- added C5: 220u, Capacitor_THT:CP_Radial_D8.0mm_P3.50mm, B.Cu at (108.3, 120.7)
- added D11: 1N4148, Diode_THT:D_DO-35_SOD27_P7.62mm_Horizontal, B.Cu at (94.0, 115.6)
- added D12: 1N4148, Diode_THT:D_DO-35_SOD27_P7.62mm_Horizontal, B.Cu at (172.7, 115.6)
- added D13: 1N4148, Diode_THT:D_DO-35_SOD27_P7.62mm_Horizontal, B.Cu at (233.7, 115.6)
- added D14: 1N4148, Diode_THT:D_DO-35_SOD27_P7.62mm_Horizontal, B.Cu at (312.4, 115.6)
- added D15: 1N4148, Diode_THT:D_DO-35_SOD27_P7.62mm_Horizontal, F.Cu at (94.0, 189.2)
- added D16: 1N4148, Diode_THT:D_DO-35_SOD27_P7.62mm_Horizontal, B.Cu at (172.7, 189.2)
- added D17: 1N4148, Diode_THT:D_DO-35_SOD27_P7.62mm_Horizontal, F.Cu at (233.7, 189.2)
- added D18: 1N4148, Diode_THT:D_DO-35_SOD27_P7.62mm_Horizontal, F.Cu at (312.4, 189.2)
- added IC1: LD1117-3.3V-SOT223, 4ms_Package_SOT:SOT223, B.Cu at (102.9, 129.5)
- added J8: USB_C_Receptacle_USB2.0_16P, Connector_USB:USB_C_Receptacle_GCT_USB4085, B.Cu at (116.4, 94.2)
- added L1: 33uH, Inductor_THT:L_Radial_D9.5mm_P5.00mm_Fastron_07HVP, B.Cu at (128.3, 106.7)
- added R11: 5.1K, Resistor_THT:R_Axial_DIN0204_L3.6mm_D1.6mm_P7.62mm_Horizontal, B.Cu at (109.2, 97.8)
- added R12: 5.1K, Resistor_THT:R_Axial_DIN0204_L3.6mm_D1.6mm_P7.62mm_Horizontal, B.Cu at (111.8, 97.8)
- added R13: 22R, Resistor_THT:R_Axial_DIN0204_L3.6mm_D1.6mm_P7.62mm_Horizontal, B.Cu at (100.3, 135.9)
- added R14: 22R, Resistor_THT:R_Axial_DIN0204_L3.6mm_D1.6mm_P7.62mm_Horizontal, B.Cu at (97.8, 135.9)
- added U5: USBLC6-2SC6, Package_TO_SOT_SMD:SOT-23-6, B.Cu at (119.4, 99.1)
- C1: value 220n -> 330u; footprint Capacitor_THT:C_Rect_L7.0mm_W4.5mm_P5.00mm -> Capacitor_THT:CP_Radial_D10.0mm_P5.00mm; moved to B.Cu
- C2, J1, R1, R4, R7, R9: moved to B.Cu
- D10: value 1N5817 -> WS2812B; footprint Diode_THT:D_DO-41_SOD81_P10.16mm_Horizontal -> LED_THT:LED_D5.0mm-4_RGB_Wide_Pins
- D2: value 1N4148 -> 1N5822; footprint Diode_THT:D_DO-35_SOD27_P7.62mm_Horizontal -> Diode_THT:D_DO-201AD_P15.24mm_Horizontal
- D3, D4, D5, D6, D7, D8: value 1N4148 -> WS2812B; footprint Diode_THT:D_DO-35_SOD27_P7.62mm_Horizontal -> LED_THT:LED_D5.0mm-4_RGB_Wide_Pins; moved to F.Cu
- D9: value 1N4148 -> WS2812B; footprint Diode_THT:D_DO-35_SOD27_P7.62mm_Horizontal -> LED_THT:LED_D5.0mm-4_RGB_Wide_Pins
- J2: value LCD -> MIDI IN; footprint midilord:4004A -> midilord:DIN5_180
- J3: value MIDI IN -> MIDI OUT 1; footprint DIN5_MIDI:DIN5_MIDI -> midilord:DIN5_180; moved to B.Cu
- J4: value MIDI OUT 1 -> MIDI OUT 2; footprint DIN5_MIDI:DIN5_MIDI -> Connector_Audio:Jack_6.35mm_Neutrik_NMJ6HFD2-AU_Horizontal; moved to B.Cu
- J5: value MIDI OUT 2 -> MIDI OUT 3; moved to B.Cu
- J6: value MIDI OUT 3 -> MIDI OUT 4; moved to B.Cu
- J7: value MIDI OUT 4 -> LCD; footprint Connector_Audio:Jack_6.35mm_Neutrik_NMJ6HFD2-AU_Horizontal -> midilord:4004A
- R10: value 1K -> 33R; moved to B.Cu
- R2: value 33R -> 1K; moved to B.Cu
- R3, R5: value 33R -> 10R; moved to B.Cu
- R6, R8: value 10R -> 33R; moved to B.Cu
- RV1: footprint Potentiometer_THT:Potentiometer_Bourns_3266W_Vertical -> Potentiometer_THT:Potentiometer_Bourns_3296Y_Vertical
- SW1, SW2, SW3, SW4, SW5, SW6, SW7, SW8: footprint Connector_PinHeader_2.54mm:PinHeader_1x02_P2.54mm_Vertical -> midilord:Footswitch; moved to F.Cu
- U1: value ESP32-S3-DevKitC -> LM2596S-5; footprint Espressif:ESP32-S3-DevKitC -> Package_TO_SOT_SMD:TO-263-5_TabPin3
- U2: value L7805 -> 6N137; footprint Package_TO_SOT_THT:TO-220-3_Vertical -> Package_DIP:DIP-8_W7.62mm; moved to B.Cu
- U3: value 6N137 -> ESP32-S3-WROOM-1; footprint Package_DIP:DIP-8_W7.62mm -> RF_Module:ESP32-S3-WROOM-1; moved to B.Cu
- moved SW5 167.9 mm to (85.1, 204.5), turned to 0 degrees
- moved SW4 165.7 mm to (321.3, 100.3), turned to 180 degrees
- moved R10 156.0 mm to (302.3, 114.3)
- moved U1 128.3 mm to (112.0, 109.2), turned to 180 degrees
- moved D3 125.7 mm to (88.3, 186.7), turned to 180 degrees
- moved U3 115.2 mm to (87.8, 155.0), turned to -90 degrees
- moved D6 110.9 mm to (324.6, 186.7), turned to 180 degrees
- moved D7 104.8 mm to (318.1, 118.1), turned to 0 degrees
- moved R9 104.7 mm to (290.8, 114.3), turned to 0 degrees
- moved J7 102.1 mm to (203.2, 152.4), turned to 0 degrees
- moved D2 96.4 mm to (118.1, 120.7), turned to 0 degrees
- moved SW7 93.2 mm to (242.6, 204.5), turned to 0 degrees
- moved SW2 92.2 mm to (163.8, 100.3), turned to 180 degrees
- moved R4 88.6 mm to (184.2, 108.0), turned to 180 degrees
- moved J2 82.7 mm to (143.6, 95.1)
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Connections:
- net MCU_MIDI_OUT4 renamed MIDI_OUT1
- C1 pad 1: Net-(D10-K) -> +9V
- C2 pad 1: +5V -> +9V
- D1 pad 1: r1 -> Net-(D1-K)
- D10 pad 1: Net-(D10-K) -> +5V
- D10 pad 2: +9V -> unconnected-(D10-DOUT-Pad2)
- D2 pad 1: r2 -> Net-(D2-K)
- D2 pad 2: Net-(D2-A) -> GND
- D3 pad 1: r1 -> +5V
- D3 pad 2: Net-(D3-A) -> Net-(D3-DOUT)
- D4 pad 1: r2 -> +5V
- D4 pad 2: Net-(D4-A) -> Net-(D4-DOUT)
- D5 pad 1: r1 -> +5V
- D5 pad 2: Net-(D5-A) -> Net-(D5-DOUT)
- D6 pad 1: r2 -> +5V
- D6 pad 2: Net-(D6-A) -> Net-(D6-DOUT)
- D7 pad 1: r1 -> +5V
- D7 pad 2: Net-(D7-A) -> Net-(D7-DOUT)
- D8 pad 1: r2 -> +5V
- D8 pad 2: Net-(D8-A) -> Net-(D8-DOUT)
- D9 pad 1: Net-(D9-K) -> +5V
- D9 pad 2: Net-(D9-A) -> Net-(D10-DIN)
- J2 pad 1: DB7 -> unconnected-(J2-Pad1)
- J2 pad 2: DB6 -> unconnected-(J2-Pad2)
- J2 pad 3: DB5 -> unconnected-(J2-Pad3)
- J2 pad 4: DB4 -> Net-(J2-Pad4)
- J2 pad 5: GND -> Net-(D1-A)
- J3 pad 2: unconnected-(J3-Pad2) -> GND
- J3 pad 5: Net-(D9-A) -> Net-(J3-Pad5)
- R1 pad 1: Net-(J3-Pad4) -> Net-(J2-Pad4)
- R1 pad 2: Net-(D9-K) -> Net-(D1-K)
- R10 pad 1: +5V -> MIDI_OUT4
- R10 pad 2: MCU_MIDI_IN -> Net-(J6-PadT)
- R2 pad 1: MCU_MIDI_OUT2 -> +5V
- R2 pad 2: Net-(J5-PadT) -> MIDI_IN
- R3 pad 1: MCU_MIDI_OUT3 -> +3.3V
- R3 pad 2: Net-(J6-PadT) -> Net-(J3-Pad4)
- R4 pad 2: Net-(J7-PadT) -> Net-(J3-Pad5)
- R5 pad 1: MCU_MIDI_OUT1 -> +3.3V
- R5 pad 2: Net-(J4-Pad5) -> Net-(J4-PadR)
- R6 pad 1: +3.3V -> MIDI_OUT2
- R6 pad 2: Net-(J5-PadR) -> Net-(J4-PadT)
- R7 pad 2: Net-(J6-PadR) -> Net-(J5-PadR)
- R8 pad 1: +3.3V -> MIDI_OUT3
- R8 pad 2: Net-(J7-PadR) -> Net-(J5-PadT)
- R9 pad 2: Net-(J4-Pad4) -> Net-(J6-PadR)
- RV1 pad 2: Net-(J2-Pin_12) -> Net-(J7-Pin_12)
- SW1 pad 1: c1 -> Net-(D11-A)
- SW1 pad 2: Net-(D1-A) -> C1
- SW2 pad 1: c1 -> Net-(D12-A)
- SW2 pad 2: Net-(D2-A) -> C2
- SW3 pad 1: c2 -> C3
- SW3 pad 2: Net-(D3-A) -> Net-(D13-A)
- SW4 pad 1: c2 -> C4
- SW4 pad 2: Net-(D4-A) -> Net-(D14-A)
- SW5 pad 1: c3 -> C1
- SW5 pad 2: Net-(D5-A) -> Net-(D15-A)
- SW6 pad 1: c3 -> C2
- SW6 pad 2: Net-(D6-A) -> Net-(D16-A)
- SW7 pad 1: c4 -> Net-(D17-A)
- SW7 pad 2: Net-(D7-A) -> C3
- SW8 pad 1: c4 -> Net-(D18-A)
- SW8 pad 2: Net-(D8-A) -> C4
- U1 pad 1: +3.3V -> +9V
- U1 pad 2: +3.3V -> Net-(D2-K)
- U1 pad 3: unconnected-(U1-CHIP_PU-Pad3) -> GND
- U1 pad 4: c3 -> +5V
- U1 pad 5: c4 -> GND
- U2 pad 1: Net-(D10-K) -> unconnected-(U2-NC-Pad1)
- U2 pad 2: GND -> Net-(D1-K)
- U2 pad 3: +5V -> Net-(D1-A)
- U3 pad 1: unconnected-(U3-NC-Pad1) -> GND
- U3 pad 2: Net-(D9-K) -> +3.3V
- U3 pad 3: Net-(D9-A) -> unconnected-(U3-EN-Pad3)
- U3 pad 5: GND -> unconnected-(U3-IO5-Pad5)
- U3 pad 6: MCU_MIDI_IN -> unconnected-(U3-IO6-Pad6)
- U3 pad 8: +5V -> unconnected-(U3-IO15-Pad8)
Routing:
- net +9V: track 0.00 -> 50.9 mm
- net Net-(J7-Pin_12): track 0.00 -> 29.6 mm
- net Net-(D2-K): track 0.00 -> 25.3 mm
- net DB4: track 0.00 -> 22.4 mm, vias 0 -> 1
- net DB6: track 0.00 -> 18.1 mm, vias 0 -> 1
- net +3.3V: track 0.00 -> 17.1 mm
- net Net-(J8-CC2): track 0.00 -> 16.4 mm
- net Net-(D1-A): track 0.00 -> 15.0 mm
- net DB7: track 0.00 -> 14.8 mm, vias 0 -> 1
- net Net-(D1-K): track 0.00 -> 14.3 mm
- net DB5: track 0.00 -> 13.3 mm, vias 0 -> 1
- net MIDI_IN: track 0.00 -> 12.8 mm
- net E2: track 0.00 -> 12.2 mm, vias 0 -> 1
- net E1: track 0.00 -> 10.7 mm, vias 0 -> 1
- net RS: track 0.00 -> 10.6 mm, vias 0 -> 1
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- added copper zone on F.Cu, net +5V
- added copper zone on In1.Cu, net GND
- added copper zone on In2.Cu, net GND
- removed copper zone on F.Cu, net GND
Other:
- board size 190.5 x 132.1 mm -> 256.5 x 129.5 mm
- copper layers 2 -> 4
- board text added: "GPIO17"

Commit message: Reduce PCB to 2-layer stackup and update design rules
Parts:
- added C6: 100n, Capacitor_THT:C_Rect_L7.0mm_W2.5mm_P5.00mm, B.Cu at (97.2, 171.4)
- added C7: 100n, Capacitor_THT:C_Rect_L7.0mm_W2.5mm_P5.00mm, B.Cu at (100.3, 171.4)
- added R15: 10K, Resistor_THT:R_Axial_DIN0204_L3.6mm_D1.6mm_P7.62mm_Horizontal, B.Cu at (94.0, 170.2)
- added R16: 10K, Resistor_THT:R_Axial_DIN0204_L3.6mm_D1.6mm_P7.62mm_Horizontal, B.Cu at (142.2, 110.5)
- added SW10: BOOT, Button_Switch_THT:SW_PUSH_1P1T_6x3.5mm_H5.0_APEM_MJTP1250, B.Cu at (83.8, 175.9)
- added SW9: RESET, Button_Switch_THT:SW_PUSH_1P1T_6x3.5mm_H5.0_APEM_MJTP1250, B.Cu at (83.8, 171.4)
- D10, D3, D4, D5, D6, D7, D8, D9: footprint LED_THT:LED_D5.0mm-4_RGB_Wide_Pins -> midilord:APA106
- D15, D17, D18, J2: moved to B.Cu
- IC1: footprint 4ms_Package_SOT:SOT223 -> Package_TO_SOT_SMD:SOT-223
- J4, J5, J6: footprint Connector_Audio:Jack_6.35mm_Neutrik_NMJ6HFD2-AU_Horizontal -> midilord:CK635-006
- moved R7 32.4 mm to (275.6, 90.2), turned to -90 degrees
- moved R5 24.3 mm to (209.6, 90.2), turned to -90 degrees
- moved R9 24.3 mm to (288.3, 90.2), turned to -90 degrees
- moved R6 15.3 mm to (209.6, 108.0), turned to 90 degrees
- moved R10 15.3 mm to (288.3, 108.0), turned to 90 degrees
- moved RV1 15.0 mm to (103.5, 176.5), turned to -90 degrees
- moved R8 12.0 mm to (275.6, 108.0), turned to 90 degrees
- moved J4 10.8 mm to (221.6, 98.4), turned to 180 degrees
- moved J5 10.8 mm to (263.5, 98.4), turned to 180 degrees
- moved J6 10.8 mm to (300.4, 98.4), turned to 180 degrees
- moved C4 1.27 mm to (94.0, 127.0)
- turned IC1 to -90 degrees
- turned J2 to 180 degrees
Connections:
- J8 pad A4: Net-(J8-VBUS-PadA4) -> unconnected-(J8-VBUS-PadA4)_2
- J8 pad A9: Net-(J8-VBUS-PadA4) -> unconnected-(J8-VBUS-PadA4)
- J8 pad B4: Net-(J8-VBUS-PadA4) -> unconnected-(J8-VBUS-PadA4)_3
- J8 pad B9: Net-(J8-VBUS-PadA4) -> unconnected-(J8-VBUS-PadA4)_1
- R2 pad 1: +5V -> +3.3V
- U2 pad 7: unconnected-(U2-EN-Pad7) -> Net-(U2-EN)
- U3 pad 22: unconnected-(U3-IO14-Pad22) -> MIDI_IN
- U3 pad 23: unconnected-(U3-IO21-Pad23) -> MIDI_OUT1
- U3 pad 24: unconnected-(U3-IO47-Pad24) -> MIDI_OUT2
- U3 pad 25: unconnected-(U3-IO48-Pad25) -> MIDI_OUT3
- U3 pad 26: unconnected-(U3-IO45-Pad26) -> MIDI_OUT4
- U3 pad 27: unconnected-(U3-IO0-Pad27) -> BOOT
- U3 pad 3: unconnected-(U3-EN-Pad3) -> RESET
- U3 pad 31: unconnected-(U3-IO38-Pad31) -> MCU_LED
- U3 pad 32: unconnected-(U3-IO39-Pad32) -> C4
- U3 pad 33: unconnected-(U3-IO40-Pad33) -> C3
- U3 pad 34: unconnected-(U3-IO41-Pad34) -> C2
- U3 pad 35: unconnected-(U3-IO42-Pad35) -> C1
- U3 pad 38: unconnected-(U3-IO2-Pad38) -> R2
- U3 pad 39: unconnected-(U3-IO1-Pad39) -> R1
Routing:
- net C4: track 0.00 -> 299.8 mm, vias 0 -> 2
- net C3: track 0.00 -> 298.4 mm, vias 0 -> 2
- net +3.3V: track 17.1 -> 300.1 mm, vias 0 -> 2
- net R1: track 0.00 -> 274.6 mm, vias 0 -> 4
- net R2: track 0.00 -> 258.1 mm
- net MIDI_OUT4: track 0.00 -> 219.1 mm
- net MIDI_OUT3: track 0.00 -> 205.7 mm
- net C2: track 0.00 -> 183.8 mm, vias 0 -> 1
- net MIDI_OUT2: track 0.00 -> 138.9 mm
- net MIDI_OUT1: track 0.00 -> 115.0 mm
- net C1: track 0.00 -> 105.4 mm, vias 0 -> 3
- net Net-(D10-DIN): track 0.00 -> 74.4 mm
- net Net-(D4-DOUT): track 0.00 -> 73.8 mm
- net Net-(D5-DOUT): track 0.00 -> 73.8 mm
- net Net-(D3-DOUT): track 0.00 -> 73.8 mm
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- removed copper zone on In1.Cu, net GND
- removed copper zone on In2.Cu, net GND
Other:
- copper layers 4 -> 2

Commit message: Add WS2812B LED support, update LCD pinout docs, and revise PCB nets
Parts:
- added C10: 100n, Capacitor_THT:C_Rect_L7.0mm_W2.5mm_P5.00mm, B.Cu at (230.5, 181.7)
- added C11: 100n, Capacitor_THT:C_Rect_L7.0mm_W2.5mm_P5.00mm, B.Cu at (309.2, 186.6)
- added C12: 100n, Capacitor_THT:C_Rect_L7.0mm_W2.5mm_P5.00mm, B.Cu at (309.2, 123.1)
- added C13: 100n, Capacitor_THT:C_Rect_L7.0mm_W2.5mm_P5.00mm, B.Cu at (230.5, 123.2)
- added C14: 100n, Capacitor_THT:C_Rect_L7.0mm_W2.5mm_P5.00mm, B.Cu at (175.9, 123.1)
- added C15: 100n, Capacitor_THT:C_Rect_L7.0mm_W2.5mm_P5.00mm, B.Cu at (78.1, 123.2)
- added C8: 100n, Capacitor_THT:C_Rect_L7.0mm_W2.5mm_P5.00mm, B.Cu at (97.2, 181.7)
- added C9: 100n, Capacitor_THT:C_Rect_L7.0mm_W2.5mm_P5.00mm, B.Cu at (175.9, 181.6)
- added JP1: LCD1, Jumper:SolderJumper-3_P1.3mm_Open_RoundedPad1.0x1.5mm, F.Cu at (102.2, 163.8)
- added JP2: LCD2, Jumper:SolderJumper-3_P1.3mm_Open_RoundedPad1.0x1.5mm, F.Cu at (102.2, 161.3)
- added JP3: LCD3, Jumper:SolderJumper-3_P1.3mm_Open_RoundedPad1.0x1.5mm, F.Cu at (102.2, 158.8)
- added JP4: LCD4, Jumper:SolderJumper-3_P1.3mm_Open_RoundedPad1.0x1.5mm, F.Cu at (102.2, 156.2)
- added JP5: LCD5, Jumper:SolderJumper-3_P1.3mm_Open_RoundedPad1.0x1.5mm, F.Cu at (102.2, 153.7)
- added JP6: LCD6, Jumper:SolderJumper-3_P1.3mm_Open_RoundedPad1.0x1.5mm, F.Cu at (102.2, 151.1)
- added JP7: LCD7, Jumper:SolderJumper-3_P1.3mm_Open_RoundedPad1.0x1.5mm, F.Cu at (102.2, 148.6)
- added JP8: LCD8, Jumper:SolderJumper-3_P1.3mm_Open_RoundedPad1.0x1.5mm, F.Cu at (102.2, 146.1)
- moved R15 10.8 mm to (83.2, 170.2), turned to 0 degrees
- moved C7 8.08 mm to (95.3, 177.8), turned to 0 degrees
- moved SW9 6.63 mm to (85.7, 177.8)
- moved C6 3.66 mm to (95.3, 174.6), turned to 0 degrees
- moved SW10 3.22 mm to (85.7, 173.4)
Connections:
- J7 pad 1: DB7 -> LCD_1
- J7 pad 2: DB6 -> LCD_2
- J7 pad 3: DB5 -> LCD_3
- J7 pad 4: DB4 -> LCD_4
- J7 pad 5: GND -> LCD_5
- J7 pad 6: GND -> LCD_6
- J7 pad 7: GND -> LCD_7
- J7 pad 8: GND -> LCD_8
- U3 pad 10: unconnected-(U3-IO17-Pad10) -> DB6
- U3 pad 11: unconnected-(U3-IO18-Pad11) -> DB5
- U3 pad 12: unconnected-(U3-IO8-Pad12) -> DB4
- U3 pad 15: DB4 -> unconnected-(U3-IO3-Pad15)
- U3 pad 16: DB6 -> unconnected-(U3-IO46-Pad16)
- U3 pad 17: DB7 -> unconnected-(U3-IO9-Pad17)
- U3 pad 18: DB5 -> unconnected-(U3-IO10-Pad18)
- U3 pad 19: E1 -> unconnected-(U3-IO11-Pad19)
- U3 pad 20: RS -> unconnected-(U3-IO12-Pad20)
- U3 pad 21: E2 -> unconnected-(U3-IO13-Pad21)
- U3 pad 6: unconnected-(U3-IO6-Pad6) -> E1
- U3 pad 7: unconnected-(U3-IO7-Pad7) -> RS
- U3 pad 8: unconnected-(U3-IO15-Pad8) -> E2
- U3 pad 9: unconnected-(U3-IO16-Pad9) -> DB7
Routing:
- net RS: track 10.6 -> 40.7 mm
- net LCD_6: track 0.00 -> 29.7 mm, vias 0 -> 2
- net LCD_2: track 0.00 -> 29.1 mm, vias 0 -> 2
- net LCD_4: track 0.00 -> 29.0 mm, vias 0 -> 2
- net LCD_1: track 0.00 -> 27.0 mm, vias 0 -> 2
- net E2: track 12.2 -> 38.7 mm
- net LCD_8: track 0.00 -> 26.3 mm
- net E1: track 10.7 -> 35.8 mm, vias 1 -> 0
- net MIDI_OUT1: track 115.0 -> 138.2 mm
- net MIDI_IN: track 77.8 -> 100.8 mm
- net MIDI_OUT2: track 138.9 -> 161.2 mm
- net MIDI_OUT3: track 205.7 -> 227.5 mm
- net MIDI_OUT4: track 219.1 -> 240.0 mm
- net LCD_3: track 0.00 -> 20.2 mm, vias 0 -> 1
- net DB7: track 13.8 -> 31.7 mm
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Other:
- board text added: "1-4"
- board text added: "5-8"
- board text added: "B"
- board text added: "D4"
- board text added: "D5"
- board text added: "D6"
- board text added: "D7"
- board text added: "E L G"
- board text added: "R"

Commit message: Add EMaj logo SVG and silkscreen artwork to PCB
Parts:
- added G***: LOGO, midilord:lain, F.Cu at (104.1, 204.5)
- added G***: LOGO, midilord:lain, B.Cu at (300.4, 204.5)
Routing:
- net RS: track 40.7 -> 39.6 mm

Commit message: Add LCD preset layout diagram and DIN5-180 connector 3D model
Parts:
- removed IC1: LD1117-3.3V-SOT223, Package_TO_SOT_SMD:SOT-223
- added G***: LOGO, midilord:emaj, F.Cu at (123.8, 204.5)
- added G***: LOGO, midilord:emaj, B.Cu at (281.3, 204.5)
- added U4: LD1117-3.3V-SOT223, Package_TO_SOT_SMD:SOT-223, B.Cu at (102.9, 129.6)
Routing:
- net Net-(D8-DOUT): track 73.3 -> 76.0 mm
- net Net-(D6-DOUT): track 70.1 -> 72.8 mm
- net Net-(D5-DOUT): track 73.8 -> 76.5 mm
- net Net-(D3-DOUT): track 73.8 -> 76.5 mm
- net Net-(D10-DIN): track 74.4 -> 77.0 mm
- net Net-(D7-DOUT): track 73.3 -> 76.0 mm
- net Net-(D4-DOUT): track 73.8 -> 76.5 mm
- net MCU_LED: track 34.1 -> 32.8 mm
Other:
- board text added: "1"
- board text added: "2"
- board text added: "3"
- board text added: "4"
- board text added: "5"
- board text added: "6"
- board text added: "7"
- board text added: "8"
- board text added: "9V"
- board text added: "MIDI IN"
- board text added: "MIDI OUT 1"
- board text added: "MIDI OUT 2"
- board text added: "MIDI OUT 3"
- board text added: "MIDI OUT 4"
- board text added: "USB"

Commit message: Add vegas mode stubs and update LED count to 8
Parts:
- moved G*** 177.8 mm to (281.9, 204.5)
- moved G*** 176.5 mm to (123.9, 204.3)
- moved G*** 0.63 mm to (124.5, 204.5)
- moved G*** 0.63 mm to (281.9, 204.5)
Other:
- board text added: "midilord"
- board text removed: "GPIO17"

Commit message: Reposition silkscreen logos, add mounting hole circles, remove channel number labels
Parts:
- moved G*** 99.5 mm to (300.4, 106.7)
- moved G*** 95.0 mm to (116.2, 109.9)
Other:
- board text removed: "1"
- board text removed: "2"
- board text removed: "3"
- board text removed: "4"
- board text removed: "5"
- board text removed: "6"
- board text removed: "7"
- board text removed: "8"
