File: hardware/core/core.kicad_sch (KiCad schematic)
At the start: 99 parts, among them J1 9V_IN, J2 MIDI IN, J3 MIDI OUT 1, J4 SWITCHES OUT, J5 EXP/AUX IN, J7 LCD, J8 USB_C_Receptacle_USB2.0_16P, J9 MIDI OUT 2/3, K1 G5V-1, K2 G5V-1, Q3 2N3904, Q4 2N3904, SW1 FS, SW10 BOOT, SW2 FS, SW3 FS, SW4 FS, SW5 FS, SW6 FS, SW7 FS, SW8 FS, SW9 RESET, U1 LM2596S-5, U2 6N137, U3 ESP32-S3-WROOM-1, U4 LD1117-3.3V-SOT223, U5 USBLC6-2SC6, U6 74HCT04

Commit message: Add switch matrix GPIO configuration and hardware updates
Parts:
- added R17: 10K, Resistor_THT:R_Axial_DIN0204_L3.6mm_D1.6mm_P7.62mm_Horizontal, symbol Device:R
Connections:
- net +3.3V: now also R17.1
- net RESET: now also R17.2
Changed lines of the file:
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@@
 	)
 	(junction
+		(at 110.49 124.46)
+		(diameter 0)
+		(color 0 0 0 0)
+	)
+	(junction
 		(at 60.96 180.34)
 		(diameter 0)
@@
 	)
 	(symbol
+		(lib_id "Device:R")
+		(at 110.49 120.65 0)
+		(unit 1)
+		(exclude_from_sim no)
+		(in_bom yes)
+		(on_board yes)
+		(dnp no)
+		(fields_autoplaced yes)
+		(property "Reference" "R17"
+			(at 113.03 119.3799 0)
+			(effects
+				(font
+					(size 1.27 1.27)
+				)
+				(justify left)
+			)
+		)
+		(property "Value" "10K"
+			(at 113.03 121.9199 0)
+			(effects
+				(font
+					(size 1.27 1.27)
+				)
+				(justify left)
+			)
+		)
+		(property "Footprint" "Resistor_THT:R_Axial_DIN0204_L3.6mm_D1.6mm_P7.62mm_Horizontal"
+			(at 108.712 120.65 90)
+			(effects
+				(font
+					(size 1.27 1.27)
+				)
+				(hide yes)
+			)
+		)
+		(property "Datasheet" "~"
+			(at 110.49 120.65 0)
+			(effects
+				(font
+					(size 1.27 1.27)
+				)
+				(hide yes)
+			)
+		)
+		(property "Description" "Resistor"
+			(at 110.49 120.65 0)
+			(effects
+				(font
+					(size 1.27 1.27)
+				)
+				(hide yes)
+			)
+		)
+		(pin "2"
+		)
+		(pin "1"
+		)
+		(instances
+			(project "core"
+				(path "/1485bec2-ae99-424e-8aed-104a9db6edd5"
+					(reference "R17")
+					(unit 1)
+				)
+			)
+		)
+	)
+	(symbol
 		(lib_id "LED:WS2812B")
 		(at 132.08 204.47 0)
@@
 					(unit 1)
 				)
+			)
+		)
+	)
+	(symbol
+		(lib_id "power:+3.3V")
+		(at 110.49 116.84 0)
+		(unit 1)
+		(exclude_from_sim no)
+		(in_bom yes)
+		(on_board yes)
+		(dnp no)
+		(fields_autoplaced yes)
+		(property "Reference" "#PWR016"
+			(at 110.49 120.65 0)
+			(effects
+				(font
+					(size 1.27 1.27)
+				)
+				(hide yes)
+			)
+		)
+		(property "Value" "+3.3V"
+			(at 110.49 111.76 0)
+			(effects
+				(font
+					(size 1.27 1.27)
+				)
+			)
+		)
+		(property "Footprint" ""
+			(at 110.49 116.84 0)
+			(effects
+				(font
+					(size 1.27 1.27)
+				)
+				(hide yes)
+			)
+		)
+		(property "Datasheet" ""
+			(at 110.49 116.84 0)
+			(effects
+				(font
+					(size 1.27 1.27)
+				)
+				(hide yes)
+			)
+		)
+		(property "Description" "Power symbol creates a global label with name \"+3.3V\""
+			(at 110.49 116.84 0)
+			(effects
+				(font
+					(size 1.27 1.27)
+				)
+				(hide yes)
+			)
+		)
+		(pin "1"
+		)
+		(instances
+			(project "core"
+				(path "/1485bec2-ae99-424e-8aed-104a9db6edd5"
+					(reference "#PWR016")
+					(unit 1)
+				)
